Commit message: + added rgbd camera joint

File: ros_robot/urdf/ros_robot.xacro (robot description, xacro)
@@ -196,3 +196,11 @@
     <dynamics damping="1.0" friction="1.0"/>
   </joint>
+  <!-- RGBD CAMERA - JOINT -->
+  <joint type="fixed" name="camera_optical_joint">
+    <origin xyz="0 0 0" rpy="-1.5707 0 -1.5707"/>
+    <child link="camera_link_optical"/>
+    <parent link="camera_link"/>
+  </joint>
+  <link name="camera_link_optical">
+  </link>
 </robot>

Commit message: + added rgbd camera to gazebo

File: ros_robot/urdf/ros_robot.xacro (robot description, xacro)
@@ -200,5 +200,5 @@
     <origin xyz="0 0 0" rpy="-1.5707 0 -1.5707"/>
     <child link="camera_link_optical"/>
-    <parent link="camera_link"/>
+    <parent link="camera"/>
   </joint>
   <link name="camera_link_optical">
